Commit message: modifications for urdfyangextension done

File: urdf/kwr75_macro.xacro (robot description, xacro)
@@ -1,11 +1,6 @@
 <?xml version="1.0"?>
 <robot name="kwr75_macro" xmlns:xacro="http://www.ros.org/wiki/xacro">
-  <xacro:macro name="kwr75_force_sensor"
-    params="
-    prefix
-    parent
-    *origin"
-  >
-    <link name="${prefix}kwr75_base_link">
+ <xacro:macro name="kwr75" params="parent id xyz:= '-1 1.2 2'">
+    <link name="kwr75_${id}_link">
       <inertial>
         <origin xyz="0.00016490924101778332 0.00015134704036161043 0.01805492934845781" rpy="0 0 0"/>
@@ -26,15 +21,91 @@
       </collision>
     </link>
-    <link name="${prefix}fts_link"/>
-    <joint name="${prefix}fts_joint" type="fixed">
-      <parent link="${prefix}kwr75_base_link" />
-      <child link="${prefix}fts_link" />
+    <link name="kwr75_${id}_fts_link"/>
+    <joint name="kwr75_${id}_fts_joint" type="fixed">
+      <parent link="kwr75_${id}_link" />
+      <child link="kwr75_${id}_fts_link" />
       <origin xyz="0 0 0.0375" rpy="0 0 0"/>
     </joint>
-    <joint name="${prefix}kwr75_base_joint" type="fixed">
+    <joint name="kwr75_${id}_joint" type="fixed">
       <parent link="${parent}" />
-      <child link="${prefix}kwr75_base_link" />
-      <xacro:insert_block name="origin" />
+      <origin xyz="${xyz}"/>
+      <child link="kwr75_${id}_link" />
     </joint>
+   <yang>
+            <!-- Radiodot network topology -->
+            <network>
+                <network-id>${L2_network_id}</network-id>
+                <supporting-network>
+                    <network-ref>${L1_network_id}</network-ref>
+                </supporting-network>
+                <node>
+                <node-id>${L2_id}</node-id>
+                <supporting-node>
+                    <network-ref>${L1_network_id}</network-ref>
+                    <node-ref>${L1_id}</node-ref>
+                </supporting-node>
+                <dl:device-layer-node-attributes xmlns:dl="urn:ietf:params:xml:ns:yang:device-layer">
+                    <dl:device-name>radiodot</dl:device-name>
+                    <dl:device-type>generic</dl:device-type>
+                </dl:device-layer-node-attributes>
+                <nt:termination-point xmlns:nt="urn:ietf:params:xml:ns:yang:ietf-network-topology">
+                    <nt:tp-id>_0</nt:tp-id>
+                    <nt:supporting-termination-point>
+                        <nt:network-ref>${L2_id}</nt:network-ref>
+                        <nt:node-ref>${L1_id}</nt:node-ref>
+                        <nt:tp-ref>eth_0</nt:tp-ref>
+                    </nt:supporting-termination-point>
+                    <dl:device-layer-termination-point-attributes xmlns:dl="urn:ietf:params:xml:ns:yang:device-layer">
+                        <dl:port-name>port1</dl:port-name>
+                        <dl:port-type>rj45</dl:port-type>
+                    </dl:device-layer-termination-point-attributes>
+                    <nl:network-layer-termination-point-attributes xmlns:nl="urn:ietf:params:xml:ns:yang:network-layer">
+                        <nl:interface-name>intf1</nl:interface-name>
+                        <nl:interface-type>ethernet</nl:interface-type>
+                        <nl:interface-status>up</nl:interface-status>
+                        <nl:mac-address>00:1A:2B:3C:4D:5E</nl:mac-address>
+                    </nl:network-layer-termination-point-attributes>
+                </nt:termination-point>
+                <nl:network-layer-node-attributes xmlns:nl="urn:ietf:params:xml:ns:yang:network-layer">
+                    <nl:node-name>netNode1</nl:node-name>
+                    <nl:node-type>generic</nl:node-type>
+                </nl:network-layer-node-attributes>
+                </node>
+                <dl:device-layer-topology xmlns:dl="urn:ietf:params:xml:ns:yang:device-layer">
+                    <dl:element>element2</dl:element>
+                </dl:device-layer-topology>
+                <nt:link xmlns:nt="urn:ietf:params:xml:ns:yang:ietf-network-topology">
+                    <nt:link-id>link1</nt:link-id>
+                    <nt:source>
+                        <nt:source-node>node1</nt:source-node>
+                        <nt:source-tp>tp1</nt:source-tp>
+                    </nt:source>
+                    <nt:destination>
+                        <nt:dest-node>node2</nt:dest-node>
+                        <nt:dest-tp>tp2</nt:dest-tp>
+                    </nt:destination>
+                    <nt:supporting-link>
+                        <nt:network-ref>network2</nt:network-ref>
+                        <nt:link-ref>link2</nt:link-ref>
+                    </nt:supporting-link>
+                    <dl:device-layer-link-attributes xmlns:dl="urn:ietf:params:xml:ns:yang:device-layer">
+                        <dl:physical-link-name>physLink1</dl:physical-link-name>
+                        <dl:physical-link-type>cat5e</dl:physical-link-type>
+                    </dl:device-layer-link-attributes>
+                    <nl:network-layer-link-attributes xmlns:nl="urn:ietf:params:xml:ns:yang:network-layer">
+                        <nl:link-name>netLink1</nl:link-name>
+                        <nl:link-type>3gpp-5g-qos-flow</nl:link-type>
+                        <nl:_5qi>1</nl:_5qi>
+                        <nl:gfbr>50</nl:gfbr>
+                        <nl:mfbr>100</nl:mfbr>
+                        <nl:pdb>20</nl:pdb>
+                        <nl:per>0</nl:per>
+                    </nl:network-layer-link-attributes>
+                </nt:link>
+                <nl:network-layer-topology xmlns:nl="urn:ietf:params:xml:ns:yang:network-layer">
+                    <nl:element>element3</nl:element>
+                </nl:network-layer-topology>
+            </network>
+        </yang>
   </xacro:macro>
 </robot>
